File: synth-hardware/keyboard/Keyboard.kicad_pcb (KiCad board)
At the start: 2 copper layers, 284.2 x 55.6 mm, 101 parts, among them J1 USB_C_Receptacle_USB2.0_16P, J2 Conn_01x04, J3 Conn_01x05, K1 SHIFT, K10 F#1, K11 G1, K12 G#1, K13 A1, K14 A#1, K15 B1, K16 C2, K17 C#2, K18 D2, K19 D#2, K2 UP, K20 E2, K21 F2, K22 F#2, K23 G2, K24 G#2, K25 A2, K26 A#2, K27 B2, K3 DOWN, K4 C1, K5 C#1, K6 D1, K7 D#1, K8 E1, K9 F1, SW2 BOOTSELECT, U1 RP2040, U2 XC6206P332MR, U3 SRV05-4, U4 W25Q128JVS, Y1 12MHz 20pF

Commit message: feat(hardware): kicad kibot workflow
Parts:
- moved FID1 21.4 mm to (71.4, 157.2)
Routing:
- net GND: track 917.9 -> 919.6 mm
Changed lines of the file:
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@@
 	(footprint "Fiducial:Fiducial_1mm_Mask2mm"
 		(layer "B.Cu")
-		(at 92.86875 157.1625 180)
+		(at 71.4375 157.1625 180)
 		(descr "Circular Fiducial, 1mm bare copper, 2mm soldermask opening (Level A)")
 		(tags "fiducial")
 		(property "Reference" "FID1"
 			(at -3.61883 -0.046823 0)
-			(layer "B.SilkS")
+			(layer "User.1")
 			(effects
 				(font
@@
 		(sheetname "Root")
 		(sheetfile "Keyboard.kicad_sch")
-		(attr smd)
+		(attr smd exclude_from_bom)
 		(fp_line
 			(start -3.11 1.785)
@@
 	)
 	(segment
+		(start 255.190625 116.284375)
+		(end 255.984375 115.490625)
+		(width 0.4)
+		(layer "B.Cu")
+		(net 7)
+	)
+	(segment
+		(start 255.984375 115.490625)
+		(end 256.512087 114.962913)
+		(width 0.4)
+		(layer "B.Cu")
+		(net 7)
+	)
+	(segment
 		(start 216.455 113.888245)
 		(end 216.955 114.388245)
@@
 	)
 	(segment
+		(start 255.984375 115.490625)
+		(end 254.79375 114.3)
+		(width 0.3)
+		(layer "B.Cu")
+		(net 7)
+	)
+	(segment
 		(start 259.907517 126.472762)
 		(end 260.187517 126.192762)
@@
 	)
 	(segment
-		(start 255.190625 116.284375)
-		(end 256.512087 114.962913)
-		(width 0.4)
-		(layer "B.Cu")
-		(net 7)
-	)
-	(segment
 		(start 233.3625 127.105622)
 		(end 236.655672 127.105622)
@@
 		(start 237.462087 114.962913)
 		(end 236.140625 116.284375)
-		(width 0.4)
+		(width 0.3)
 		(layer "B.Cu")
 		(net 7)
@@
 		(start 239.38131 111.684041)
 		(end 258.425425 111.684041)
-		(width 0.4)
+		(width 0.3)
 		(layer "F.Cu")
 		(net 10)
@@
 		(start 238.116161 112.94919)
 		(end 239.38131 111.684041)
-		(width 0.4)
+		(width 0.3)
 		(layer "B.Cu")
 		(net 10)
