File: synth-hardware/keyboard/Keyboard.kicad_sch (KiCad schematic)
At the start: 101 parts, among them J1 USB_C_Receptacle_USB2.0_16P, J2 Conn_01x04, J3 Conn_01x05, K1 SHIFT, K10 F#1, K11 G1, K12 G#1, K13 A1, K14 A#1, K15 B1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

Commit message: feat(hardware): kicad kibot workflow
Parts:
- J2: now left out of the parts list
Changed lines of the file:
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@@
 		(unit 1)
 		(exclude_from_sim no)
-		(in_bom yes)
+		(in_bom no)
 		(on_board yes)
 		(dnp no)
